Commit message: transform robot into quadruped

File: body.urdf (robot description, URDF)
Before this commit: robot robot, 3 links, 2 joints
Links:
- added link Back_Lower_Leg, mass 1; collision box size=0.2 0.2 1.0; visual box size=0.2 0.2 1.0
- added link Front_Lower_Leg, mass 1; collision box size=0.2 0.2 1.0; visual box size=0.2 0.2 1.0
- added link Left_Leg, mass 1; collision box size=1.0 0.2 0.2; visual box size=1.0 0.2 0.2
- added link Left_Lower_Leg, mass 1; collision box size=0.2 0.2 1.0; visual box size=0.2 0.2 1.0
- added link Right_Leg, mass 1; collision box size=1.0 0.2 0.2; visual box size=1.0 0.2 0.2
- added link Right_Lower_Leg, mass 1; collision box size=0.2 0.2 1.0; visual box size=0.2 0.2 1.0
- link Back_Leg: geometry collision box size=0.2 1.0 0.2; visual box size=0.2 1.0 0.2
- link Front_Leg: geometry collision box size=0.2 1.0 0.2; visual box size=0.2 1.0 0.2
Joints:
- added joint Back_Lower_Leg_Joint: type revolute, parent Back_Leg, child Back_Lower_Leg, origin xyz=0.0 -1.0 0.0 rpy=0 0 0, axis 1 0 0, limit lower=-3.14159 upper=3.14159 effort=0.0 velocity=0.0
- added joint Front_Lower_Leg_Joint: type revolute, parent Front_Leg, child Front_Lower_Leg, origin xyz=0.0 1.0 0.0 rpy=0 0 0, axis 1 0 0, limit lower=-3.14159 upper=3.14159 effort=0.0 velocity=0.0
- added joint Left_Lower_Leg_Joint: type revolute, parent Left_Leg, child Left_Lower_Leg, origin xyz=-1.0 0.0 0.0 rpy=0 0 0, axis 1 0 0, limit lower=-3.14159 upper=3.14159 effort=0.0 velocity=0.0
- added joint Right_Lower_Leg_Joint: type revolute, parent Right_Leg, child Right_Lower_Leg, origin xyz=1.0 0.0 0.0 rpy=0 0 0, axis 1 0 0, limit lower=-3.14159 upper=3.14159 effort=0.0 velocity=0.0
- added joint Torso_Left_Leg: type revolute, parent Torso, child Left_Leg, origin xyz=-0.5 0.0 1.0 rpy=0 0 0, axis 1 0 0, limit lower=-3.14159 upper=3.14159 effort=0.0 velocity=0.0
- added joint Torso_Right_Leg: type revolute, parent Torso, child Right_Leg, origin xyz=0.5 0.0 1.0 rpy=0 0 0, axis 1 0 0, limit lower=-3.14159 upper=3.14159 effort=0.0 velocity=0.0
- joint Torso_Back_Leg: axis 0 1 0 -> 1 0 0; origin xyz=1.0 0.0 1.0 rpy=0 0 0 -> xyz=0.0 -0.5 1.0 rpy=0 0 0
- joint Torso_Front_Leg: axis 0 1 0 -> 1 0 0; origin xyz=2.0 0.0 1.0 rpy=0 0 0 -> xyz=0.0 0.5 1.0 rpy=0 0 0

Commit message: change vectors of legs

File: body.urdf (robot description, URDF)
Before this commit: robot robot, 9 links, 8 joints
Joints:
- joint Left_Lower_Leg_Joint: axis 1 0 0 -> 0 1 0
- joint Right_Lower_Leg_Joint: axis 1 0 0 -> 0 1 0
- joint Torso_Left_Leg: axis 1 0 0 -> 0 1 0
- joint Torso_Right_Leg: axis 1 0 0 -> 0 1 0
